Commit message: compile

File: tetra_description/urdf/base.urdf.xacro (robot description, xacro)
@@ -1,4 +1,4 @@
 <?xml version="1.0"?>
-<robot name="tetraDS" xmlns:xacro="http://ros.org/wiki/xacro">
+<robot name="tetra" xmlns:xacro="http://www.ros.org/wiki/xacro">
   <!-- Define a number of dimensions using properties -->
   <xacro:property name="base_length" value="0.473" />
@@ -24,7 +24,7 @@
     <origin xyz=" 0 ${-1.0*wheel_offset_y} 0 " rpy="0 0 0" />
 	<geometry>
-	  <mesh filename="package://tetra_description/meshes/Wheel Drive Left.STL" scale="0.001 0.001 0.001" />
+	  <mesh filename="package://tetra_description/meshes/wheel_drive_left.stl" scale="0.001 0.001 0.001" />
 	</geometry>
-	<material name="DarkGrey"/>
+	<material name="darkgrey"/>
   </visual>
     </link>
@@ -39,19 +39,18 @@
     <origin xyz=" 0 ${wheel_offset_y} 0 " rpy="0 0 0" />
 	<geometry>
-	  <mesh filename="package://tetra_description/meshes/Wheel Drive Right.STL" scale="0.001 0.001 0.001" />
+	  <mesh filename="package://tetra_description/meshes/wheel_drive_right.stl" scale="0.001 0.001 0.001" />
 	</geometry>
-	<material name="DarkGrey"/>
+	<material name="darkgrey"/>
   </visual>
     </link>
   <!-- The base xacro macro -->
-  <xacro:macro name="base" params="name color">
-   <link name="${name}_link">
+   <link name="base_link">
     <visual>
     <origin xyz=" 0 0 0 " rpy="0 0 0" />
       <geometry>
         <mesh
-          filename="package://tetra_description/meshes/Platform Body_L.STL" scale="0.001 0.001 0.001" />
+          filename="package://tetra_description/meshes/platform_body_l.stl" scale="0.001 0.001 0.001" />
       </geometry>
-      <material name="Black"/>
+      <material name="black"/>
     </visual>
       <collision>
@@ -62,5 +61,4 @@
       </collision>
     </link>
-  </xacro:macro>
   <link name="base_footprint">
       <visual>
@@ -69,5 +67,5 @@
 	  <box size="0.641 0.490 0.001" />
         </geometry>
-        <material name="TransparentGreen" />
+        <material name="transparentgreen" />
       </visual>
   </link>
@@ -83,12 +81,12 @@
                 <origin xyz="0 0 0" rpy="0 0 0"/>
                 <geometry>
-                    <mesh filename="package://tetra_description/meshes/Caster Yoke.STL" scale="0.001 0.001 0.001" />
+                    <mesh filename="package://tetra_description/meshes/caster_yoke.stl" scale="0.001 0.001 0.001" />
                 </geometry>
-                <material name="DarkGrey" />
+                <material name="darkgrey" />
             </visual>
             <collision>
                 <origin xyz="0 0 0" rpy="0 0 0"/>
                 <geometry>
-                    <mesh filename="package://tetra_description/meshes/Caster Yoke.STL" scale="0.001 0.001 0.001" />
+                    <mesh filename="package://tetra_description/meshes/caster_yoke.stl" scale="0.001 0.001 0.001" />
                 </geometry>
             </collision>
@@ -109,12 +107,12 @@
                 <origin xyz="0 0 0" rpy="0 0 0"/>
                 <geometry>
-                    <mesh filename="package://tetra_description/meshes/Caster Wheel.STL" scale="0.001 0.001 0.001" />
+                    <mesh filename="package://tetra_description/meshes/caster_wheel.stl" scale="0.001 0.001 0.001" />
                 </geometry>
-                <material name="DarkGrey" />
+                <material name="darkgrey" />
             </visual>
             <collision>
                 <origin xyz="0 0 0" rpy="0 0 0"/>
                 <geometry>
-                    <mesh filename="package://tetra_description/meshes/Caster Wheel.STL" scale="0.001 0.001 0.001" />
+                    <mesh filename="package://tetra_description/meshes/caster_wheel.stl" scale="0.001 0.001 0.001" />
                 </geometry>
             </collision>

File: tetra_description/urdf/materials.urdf.xacro (robot description, xacro)
@@ -2,44 +2,44 @@
 <robot>
   <!-- Put all the color definitions in a separate file -->
-  <material name="Black">
+  <material name="black">
     <color rgba="0.2 0.2 0.2 1.0"/>
   </material>
-   <material name="TransparentBlack">
+   <material name="transparentblack">
     <color rgba="0.2 0.2 0.2 1.0"/>
   </material>
-  <material name="Orange">
+  <material name="orange">
     <color rgba="1.0  0.55 0.0 1.0"/>
   </material>
-  <material name="Grey">
+  <material name="grey">
     <color rgba="0.7 0.7 0.7 1.0"/>
   </material>
-  <material name="DarkGrey">
+  <material name="darkgrey">
     <color rgba="0.4 0.4 0.4 1.0"/>
   </material>
-  <material name="Red">
+  <material name="red">
     <color rgba="0.8 0.0 0.0 1.0"/>
   </material>
-  <material name="TransparentRed">
+  <material name="transparentred">
     <color rgba="0.5 0.1 0.1 1.0"/>
   </material>
-  <material name="White">
+  <material name="white">
     <color rgba="1.0 1.0 1.0 0.98"/>
   </material>
-  <material name="OffWhite">
+  <material name="offWhite">
     <color rgba="0.8 0.8 0.8 1.0"/>
   </material>
-  <material name="Blue">
+  <material name="blue">
     <color rgba="0.0 0.0 0.8 1.0"/>
   </material>
-  <material name="Green">
+  <material name="green">
     <color rgba="0.0 0.8 0.0 1.0"/>
   </material>
-  <material name="TransparentGreen">
+  <material name="transparentgreen">
     <color rgba="0.0 0.8 0.0 0.5"/>
   </material>
- <material name="TransparentBlue">
+ <material name="transparentblue">
     <color rgba="0.0 0.0 0.6 0.8"/>
   </material>
- <material name="TransparentYellow">
+ <material name="transparentyellow">
     <color rgba="0.8 0.8 0.1 1.0"/>
   </material>

File: tetra_description/urdf/tetraDS.xacro (robot description, xacro)
@@ -1,4 +1,4 @@
 <?xml version="1.0"?>
-<robot name="tetraDS" xmlns:xacro="http://ros.org/wiki/xacro">
+<robot name="tetra" xmlns:xacro="http://www.ros.org/wiki/xacro">
   <!-- Define a number of dimensions using properties -->
   <xacro:property name="base_length" value="0.473" />
@@ -7,31 +7,12 @@
   <xacro:property name="wheel_radius" value="0.085" />
   <xacro:property name="wheel_offset_x" value="0.0" />
-  <xacro:property name="wheel_offset_y" value="0.207" /> <!--0.220-->
+  <xacro:property name="wheel_offset_y" value="0.207" />
   <xacro:property name="wheel_offset_z" value="-0.100" />
   <xacro:property name="PI" value="3.1415926" />
-  <xacro:macro name="cylinder_inertia" params="m r h">
-        <inertia ixx="${m*(3*r*r+h*h)/12}" ixy="0" ixz="0" iyy="${m*(3*r*r+h*h)/12}" iyz="0" izz="${m*r*r/2}" />
-  </xacro:macro>
-   <!-- Include all component files -->
-   <xacro:include filename="$(find tetra_description)/urdf/materials.urdf.xacro" />
-   <xacro:include filename="$(find tetra_description)/urdf/base.urdf.xacro" />
-   <!-- Add the base and wheels -->
-   <base name="base" color="Black"/>
-  <link name="base_link">
-    <visual>
-    <origin xyz=" 0 0 0 " rpy="0 0 0" />
-      <geometry>
-        <mesh
-          filename="package://tetra_description/meshes/Platform Body_L.STL" scale="0.001 0.001 0.001" />
-      </geometry>
-      <material name="Black"/>
-    </visual>
-      <collision>
-            <origin xyz="0 0 0" rpy="0 0 0"/>
-            <geometry>
-                <cylinder length="${base_length}" radius="${base_radius}"/>
-            </geometry>
-      </collision>
-    </link>
+  <!-- Include all component files -->
+  <xacro:include filename="$(find tetra_description)/urdf/materials.urdf.xacro" />
+  <xacro:include filename="$(find tetra_description)/urdf/base.urdf.xacro" />
+  <!-- Add the base and wheels -->
+  <!--<base name="base" color="Black"/>-->
   <link name="laser">
       <visual>
@@ -40,5 +21,5 @@
           <box size="0.01 0.01 0.01" />
         </geometry>
-        <material name="Grey" />
+        <material name="grey" />
       </visual>
   </link>
@@ -48,18 +29,4 @@
     <child link="laser" />
   </joint>
-  <link name="laser_link2">
-      <visual>
-        <origin xyz="0 0 0" rpy="0 0 0" />
-        <geometry>
-          <box size="0.01 0.01 0.01" />
-        </geometry>
-        <material name="Grey" />
-      </visual>
-  </link>
-  <joint name="base_link_to_laser_link2" type="fixed">
-    <origin xyz="-0.390 0.0 0.211" rpy="0 0 ${PI}" />
-    <parent link="base_link"/>
-    <child link="laser_link2" />
-  </joint>
   <link name="imu_link">
       <visual>
@@ -68,5 +35,5 @@
           <box size="0.01 0.01 0.01" />
         </geometry>
-        <material name="Grey" />
+        <material name="grey" />
       </visual>
   </link>
@@ -82,13 +49,13 @@
           <box size="0.01 0.01 0.01" />
         </geometry>
-        <material name="Grey" />
+        <material name="grey" />
       </visual>
   </link>
   <joint name="usb_cam" type="fixed">
-    <origin xyz="-0.384 0.0 0.1817" rpy="1.5708 3.14159 4.71239"/>
+    <origin xyz="-0.384 0.0 0.1387" rpy="1.5708 3.14159 4.71239"/>
     <parent link="base_link"/>
     <child link="usb_cam" />
   </joint>
- <link name="Front_bumper">
+ <link name="front_bumper">
       <visual>
         <origin xyz="0 0 0" rpy="0 0 0" />
@@ -96,11 +63,11 @@
           <box size="0.01 0.48 0.01" />
         </geometry>
-        <material name="TransparentBlack" />
+        <material name="transparentblack" />
       </visual>
   </link>
-  <joint name="Front_bumper" type="fixed">
+  <joint name="front_bumper" type="fixed">
     <origin xyz="0.2 0.0 -0.05" rpy="0 0 0" />
     <parent link="base_link"/>
-    <child link="Front_bumper" />
+    <child link="front_bumper" />
   </joint>
  <link name="camera1_link">
@@ -110,14 +77,14 @@
           <box size="0.01 0.01 0.01" />
         </geometry>
-        <material name="Grey" />
+        <material name="grey" />
       </visual>
   </link>
   <joint name="camera1_link" type="fixed">
     <!--<origin xyz="0.1553 -0.1155 0.0" rpy="3.14 -0.261799 0" />-->
-    <origin xyz="0.1553 0.0 0.0" rpy="0 0 0" />
+    <origin xyz="0.1553 0.079 0.0" rpy="0 0 0" />
     <parent link="base_link"/>
     <child link="camera1_link" />
   </joint>
-   <link name="camera2_link">
+ <link name="camera2_link">
       <visual>
         <origin xyz="0 0 0" rpy="0 0 0" />
@@ -125,21 +92,20 @@
           <box size="0.01 0.01 0.01" />
         </geometry>
-        <material name="Grey" />
+        <material name="grey" />
       </visual>
   </link>
   <joint name="camera2_link" type="fixed">
-    <!--<origin xyz="0.1553 -0.1155 0.0" rpy="3.14 -0.261799 0" />-->
-    <origin xyz="0.1553 0.0 0.0" rpy="0 0 0" />
+    <origin xyz="0.1553 -0.1145 0.0" rpy="0 0 0" />
     <parent link="base_link"/>
     <child link="camera2_link" />
   </joint>
- <link name="base_Upperlink">
+ <link name="base_upperlink">
    <visual>
     <origin xyz=" 0 0 0 " rpy="0 0 0" />
       <geometry>
         <mesh
-          filename="package://tetra_description/meshes/Platform Body_U.STL" scale="0.001 0.001 0.001" />
+          filename="package://tetra_description/meshes/platform_body_u.stl" scale="0.001 0.001 0.001" />
       </geometry>
-      <material name="TransparentRed"/>
+      <material name="transparentred"/>
     </visual>
       <collision>
@@ -150,8 +116,8 @@
       </collision>
   </link>
-  <joint name="base_Upperlink" type="fixed">
+  <joint name="base_upperlink" type="fixed">
     <origin xyz="0.0 0.0 0.0" rpy="0 0 0" />
     <parent link="base_link"/>
-    <child link="base_Upperlink" />
+    <child link="base_upperlink" />
   </joint>
 </robot>

Commit message: frame name adjust

File: tetra_description/urdf/base.urdf.xacro (robot description, xacro)
@@ -1,4 +1,4 @@
 <?xml version="1.0"?>
-<robot name="tetra" xmlns:xacro="http://www.ros.org/wiki/xacro">
+<robot name="tetraDS" xmlns:xacro="http://ros.org/wiki/xacro">
   <!-- Define a number of dimensions using properties -->
   <xacro:property name="base_length" value="0.473" />
@@ -24,7 +24,7 @@
     <origin xyz=" 0 ${-1.0*wheel_offset_y} 0 " rpy="0 0 0" />
 	<geometry>
-	  <mesh filename="package://tetra_description/meshes/wheel_drive_left.stl" scale="0.001 0.001 0.001" />
+	  <mesh filename="package://tetra_description/meshes/Wheel Drive Left.STL" scale="0.001 0.001 0.001" />
 	</geometry>
-	<material name="darkgrey"/>
+	<material name="DarkGrey"/>
   </visual>
     </link>
@@ -39,18 +39,19 @@
     <origin xyz=" 0 ${wheel_offset_y} 0 " rpy="0 0 0" />
 	<geometry>
-	  <mesh filename="package://tetra_description/meshes/wheel_drive_right.stl" scale="0.001 0.001 0.001" />
+	  <mesh filename="package://tetra_description/meshes/Wheel Drive Right.STL" scale="0.001 0.001 0.001" />
 	</geometry>
-	<material name="darkgrey"/>
+	<material name="DarkGrey"/>
   </visual>
     </link>
   <!-- The base xacro macro -->
-   <link name="base_link">
+  <xacro:macro name="base" params="name color">
+   <link name="${name}_link">
     <visual>
     <origin xyz=" 0 0 0 " rpy="0 0 0" />
       <geometry>
         <mesh
-          filename="package://tetra_description/meshes/platform_body_l.stl" scale="0.001 0.001 0.001" />
+          filename="package://tetra_description/meshes/Platform Body_L.STL" scale="0.001 0.001 0.001" />
       </geometry>
-      <material name="black"/>
+      <material name="Black"/>
     </visual>
       <collision>
@@ -61,4 +62,5 @@
       </collision>
     </link>
+  </xacro:macro>
   <link name="base_footprint">
       <visual>
@@ -67,5 +69,5 @@
 	  <box size="0.641 0.490 0.001" />
         </geometry>
-        <material name="transparentgreen" />
+        <material name="TransparentGreen" />
       </visual>
   </link>
@@ -81,12 +83,12 @@
                 <origin xyz="0 0 0" rpy="0 0 0"/>
                 <geometry>
-                    <mesh filename="package://tetra_description/meshes/caster_yoke.stl" scale="0.001 0.001 0.001" />
+                    <mesh filename="package://tetra_description/meshes/Caster Yoke.STL" scale="0.001 0.001 0.001" />
                 </geometry>
-                <material name="darkgrey" />
+                <material name="DarkGrey" />
             </visual>
             <collision>
                 <origin xyz="0 0 0" rpy="0 0 0"/>
                 <geometry>
-                    <mesh filename="package://tetra_description/meshes/caster_yoke.stl" scale="0.001 0.001 0.001" />
+                    <mesh filename="package://tetra_description/meshes/Caster Yoke.STL" scale="0.001 0.001 0.001" />
                 </geometry>
             </collision>
@@ -107,12 +109,12 @@
                 <origin xyz="0 0 0" rpy="0 0 0"/>
                 <geometry>
-                    <mesh filename="package://tetra_description/meshes/caster_wheel.stl" scale="0.001 0.001 0.001" />
+                    <mesh filename="package://tetra_description/meshes/Caster Wheel.STL" scale="0.001 0.001 0.001" />
                 </geometry>
-                <material name="darkgrey" />
+                <material name="DarkGrey" />
             </visual>
             <collision>
                 <origin xyz="0 0 0" rpy="0 0 0"/>
                 <geometry>
-                    <mesh filename="package://tetra_description/meshes/caster_wheel.stl" scale="0.001 0.001 0.001" />
+                    <mesh filename="package://tetra_description/meshes/Caster Wheel.STL" scale="0.001 0.001 0.001" />
                 </geometry>
             </collision>

File: tetra_description/urdf/materials.urdf.xacro (robot description, xacro)
@@ -2,44 +2,44 @@
 <robot>
   <!-- Put all the color definitions in a separate file -->
-  <material name="black">
+  <material name="Black">
     <color rgba="0.2 0.2 0.2 1.0"/>
   </material>
-   <material name="transparentblack">
+   <material name="TransparentBlack">
     <color rgba="0.2 0.2 0.2 1.0"/>
   </material>
-  <material name="orange">
+  <material name="Orange">
     <color rgba="1.0  0.55 0.0 1.0"/>
   </material>
-  <material name="grey">
+  <material name="Grey">
     <color rgba="0.7 0.7 0.7 1.0"/>
   </material>
-  <material name="darkgrey">
+  <material name="DarkGrey">
     <color rgba="0.4 0.4 0.4 1.0"/>
   </material>
-  <material name="red">
+  <material name="Red">
     <color rgba="0.8 0.0 0.0 1.0"/>
   </material>
-  <material name="transparentred">
+  <material name="TransparentRed">
     <color rgba="0.5 0.1 0.1 1.0"/>
   </material>
-  <material name="white">
+  <material name="White">
     <color rgba="1.0 1.0 1.0 0.98"/>
   </material>
-  <material name="offWhite">
+  <material name="OffWhite">
     <color rgba="0.8 0.8 0.8 1.0"/>
   </material>
-  <material name="blue">
+  <material name="Blue">
     <color rgba="0.0 0.0 0.8 1.0"/>
   </material>
-  <material name="green">
+  <material name="Green">
     <color rgba="0.0 0.8 0.0 1.0"/>
   </material>
-  <material name="transparentgreen">
+  <material name="TransparentGreen">
     <color rgba="0.0 0.8 0.0 0.5"/>
   </material>
- <material name="transparentblue">
+ <material name="TransparentBlue">
     <color rgba="0.0 0.0 0.6 0.8"/>
   </material>
- <material name="transparentyellow">
+ <material name="TransparentYellow">
     <color rgba="0.8 0.8 0.1 1.0"/>
   </material>

File: tetra_description/urdf/tetraDS.xacro (robot description, xacro)
@@ -1,4 +1,4 @@
 <?xml version="1.0"?>
-<robot name="tetra" xmlns:xacro="http://www.ros.org/wiki/xacro">
+<robot name="tetraDS" xmlns:xacro="http://ros.org/wiki/xacro">
   <!-- Define a number of dimensions using properties -->
   <xacro:property name="base_length" value="0.473" />
@@ -7,12 +7,15 @@
   <xacro:property name="wheel_radius" value="0.085" />
   <xacro:property name="wheel_offset_x" value="0.0" />
-  <xacro:property name="wheel_offset_y" value="0.207" />
+  <xacro:property name="wheel_offset_y" value="0.207" /> <!--0.220-->
   <xacro:property name="wheel_offset_z" value="-0.100" />
   <xacro:property name="PI" value="3.1415926" />
-  <!-- Include all component files -->
-  <xacro:include filename="$(find tetra_description)/urdf/materials.urdf.xacro" />
-  <xacro:include filename="$(find tetra_description)/urdf/base.urdf.xacro" />
-  <!-- Add the base and wheels -->
-  <!--<base name="base" color="Black"/>-->
+  <xacro:macro name="cylinder_inertia" params="m r h">
+        <inertia ixx="${m*(3*r*r+h*h)/12}" ixy="0" ixz="0" iyy="${m*(3*r*r+h*h)/12}" iyz="0" izz="${m*r*r/2}" />
+  </xacro:macro>
+   <!-- Include all component files -->
+   <xacro:include filename="$(find tetra_description)/urdf/materials.urdf.xacro" />
+   <xacro:include filename="$(find tetra_description)/urdf/base.urdf.xacro" />
+   <!-- Add the base and wheels -->
+   <base name="base" color="Black"/>
   <link name="laser">
       <visual>
@@ -21,5 +24,5 @@
           <box size="0.01 0.01 0.01" />
         </geometry>
-        <material name="grey" />
+        <material name="Grey" />
       </visual>
   </link>
@@ -29,4 +32,18 @@
     <child link="laser" />
   </joint>
+  <link name="laser_link2">
+      <visual>
+        <origin xyz="0 0 0" rpy="0 0 0" />
+        <geometry>
+          <box size="0.01 0.01 0.01" />
+        </geometry>
+        <material name="Grey" />
+      </visual>
+  </link>
+  <joint name="base_link_to_laser_link2" type="fixed">
+    <origin xyz="-0.390 0.0 0.211" rpy="0 0 ${PI}" />
+    <parent link="base_link"/>
+    <child link="laser_link2" />
+  </joint>
   <link name="imu_link">
       <visual>
@@ -35,5 +52,5 @@
           <box size="0.01 0.01 0.01" />
         </geometry>
-        <material name="grey" />
+        <material name="Grey" />
       </visual>
   </link>
@@ -49,13 +66,13 @@
           <box size="0.01 0.01 0.01" />
         </geometry>
-        <material name="grey" />
+        <material name="Grey" />
       </visual>
   </link>
   <joint name="usb_cam" type="fixed">
-    <origin xyz="-0.384 0.0 0.1387" rpy="1.5708 3.14159 4.71239"/>
+    <origin xyz="-0.384 0.0 0.1817" rpy="1.5708 3.14159 4.71239"/>
     <parent link="base_link"/>
     <child link="usb_cam" />
   </joint>
- <link name="front_bumper">
+ <link name="Front_bumper">
       <visual>
         <origin xyz="0 0 0" rpy="0 0 0" />
@@ -63,11 +80,11 @@
           <box size="0.01 0.48 0.01" />
         </geometry>
-        <material name="transparentblack" />
+        <material name="TransparentBlack" />
       </visual>
   </link>
-  <joint name="front_bumper" type="fixed">
+  <joint name="Front_bumper" type="fixed">
     <origin xyz="0.2 0.0 -0.05" rpy="0 0 0" />
     <parent link="base_link"/>
-    <child link="front_bumper" />
+    <child link="Front_bumper" />
   </joint>
  <link name="camera1_link">
@@ -77,14 +94,14 @@
           <box size="0.01 0.01 0.01" />
         </geometry>
-        <material name="grey" />
+        <material name="Grey" />
       </visual>
   </link>
   <joint name="camera1_link" type="fixed">
     <!--<origin xyz="0.1553 -0.1155 0.0" rpy="3.14 -0.261799 0" />-->
-    <origin xyz="0.1553 0.079 0.0" rpy="0 0 0" />
+    <origin xyz="0.1553 0.0 0.0" rpy="0 0 0" />
     <parent link="base_link"/>
     <child link="camera1_link" />
   </joint>
- <link name="camera2_link">
+   <link name="camera2_link">
       <visual>
         <origin xyz="0 0 0" rpy="0 0 0" />
@@ -92,20 +109,21 @@
           <box size="0.01 0.01 0.01" />
         </geometry>
-        <material name="grey" />
+        <material name="Grey" />
       </visual>
   </link>
   <joint name="camera2_link" type="fixed">
-    <origin xyz="0.1553 -0.1145 0.0" rpy="0 0 0" />
+    <!--<origin xyz="0.1553 -0.1155 0.0" rpy="3.14 -0.261799 0" />-->
+    <origin xyz="0.1553 0.0 0.0" rpy="0 0 0" />
     <parent link="base_link"/>
     <child link="camera2_link" />
   </joint>
- <link name="base_upperlink">
+ <link name="base_Upperlink">
    <visual>
     <origin xyz=" 0 0 0 " rpy="0 0 0" />
       <geometry>
         <mesh
-          filename="package://tetra_description/meshes/platform_body_u.stl" scale="0.001 0.001 0.001" />
+          filename="package://tetra_description/meshes/Platform Body_U.STL" scale="0.001 0.001 0.001" />
       </geometry>
-      <material name="transparentred"/>
+      <material name="TransparentRed"/>
     </visual>
       <collision>
@@ -116,8 +134,8 @@
       </collision>
   </link>
-  <joint name="base_upperlink" type="fixed">
+  <joint name="base_Upperlink" type="fixed">
     <origin xyz="0.0 0.0 0.0" rpy="0 0 0" />
     <parent link="base_link"/>
-    <child link="base_upperlink" />
+    <child link="base_Upperlink" />
   </joint>
 </robot>
